Commit message: Milestone 4: Add 2D LiDAR sensor and LaserScan support

File: src/warehouse_robot_description/urdf/gazebo.xacro (robot description, xacro)
@@ -13,4 +13,12 @@
   <gazebo reference="caster_wheel">
     <material>Gazebo/Grey</material>
+  </gazebo>
+    <!-- Gazebo Sensors System -->
+  <gazebo>
+    <plugin
+      filename="gz-sim-sensors-system"
+      name="gz::sim::systems::Sensors">
+      <render_engine>ogre2</render_engine>
+    </plugin>
   </gazebo>
   <!-- Differential Drive Plugin -->
@@ -29,3 +37,27 @@
     </plugin>
   </gazebo>
+    <!-- ================= LiDAR Sensor ================= -->
+  <gazebo reference="lidar_link">
+    <sensor name="lidar_sensor" type="gpu_lidar">
+      <update_rate>10</update_rate>
+      <topic>scan</topic>
+      <lidar>
+        <scan>
+          <horizontal>
+            <samples>720</samples>
+            <resolution>1</resolution>
+            <min_angle>-3.14159</min_angle>
+            <max_angle>3.14159</max_angle>
+          </horizontal>
+        </scan>
+        <range>
+          <min>0.12</min>
+          <max>10.0</max>
+          <resolution>0.01</resolution>
+        </range>
+      </lidar>
+      <always_on>true</always_on>
+      <visualize>true</visualize>
+    </sensor>
+  </gazebo>
 </robot>

File: src/warehouse_robot_description/urdf/warehouse_robot.urdf.xacro (robot description, xacro)
@@ -2,4 +2,5 @@
 <robot xmlns:xacro="http://www.ros.org/wiki/xacro"
        name="warehouse_robot">
+  <xacro:include filename="$(find warehouse_robot_description)/urdf/gazebo.xacro"/>
   <!-- Robot Dimensions -->
   <xacro:property name="robot_length" value="0.40"/>
@@ -8,4 +9,7 @@
   <xacro:property name="wheel_radius" value="0.05"/>
   <xacro:property name="wheel_width" value="0.03"/>
+  <!-- LiDAR dimensions -->
+<xacro:property name="lidar_radius" value="0.04"/>
+<xacro:property name="lidar_height" value="0.05"/>
   <!-- ================= BASE ================= -->
   <link name="base_link">
@@ -35,4 +39,31 @@
     </inertial>
   </link>
+  <!-- ================= LiDAR ================= -->
+<link name="lidar_link">
+  <visual>
+    <geometry>
+      <cylinder radius="${lidar_radius}" length="${lidar_height}"/>
+    </geometry>
+    <material name="Black">
+      <color rgba="0.2 0.2 0.2 1"/>
+    </material>
+  </visual>
+  <collision>
+    <geometry>
+      <cylinder radius="${lidar_radius}" length="${lidar_height}"/>
+    </geometry>
+  </collision>
+  <inertial>
+    <mass value="0.2"/>
+    <origin xyz="0 0 0"/>
+    <inertia
+      ixx="0.0001"
+      ixy="0"
+      ixz="0"
+      iyy="0.0001"
+      iyz="0"
+      izz="0.0001"/>
+  </inertial>
+</link>
   <!-- ================= LEFT WHEEL ================= -->
   <link name="left_wheel">
@@ -152,4 +183,13 @@
           rpy="0 0 0"/>
   </joint>
-  <xacro:include filename="gazebo.xacro"/>
+  <!-- ================= LiDAR JOINT ================= -->
+<joint
+    name="lidar_joint"
+    type="fixed">
+    <parent link="base_link"/>
+    <child link="lidar_link"/>
+    <origin
+        xyz="0 0 0.10"
+        rpy="0 0 0"/>
+</joint>
 </robot>

Commit message: Milestone 5: Add RGB camera sensor and ROS image streaming

File: src/warehouse_robot_description/urdf/gazebo.xacro (robot description, xacro)
@@ -61,3 +61,24 @@
     </sensor>
   </gazebo>
+    <!-- ================= Camera Sensor ================= -->
+  <gazebo reference="camera_link">
+    <sensor name="camera_sensor" type="camera">
+      <always_on>true</always_on>
+      <update_rate>30</update_rate>
+      <visualize>true</visualize>
+      <topic>camera</topic>
+      <camera>
+        <horizontal_fov>1.3962634</horizontal_fov>
+        <image>
+          <width>640</width>
+          <height>480</height>
+          <format>R8G8B8</format>
+        </image>
+        <clip>
+          <near>0.1</near>
+          <far>100</far>
+        </clip>
+      </camera>
+    </sensor>
+  </gazebo>
 </robot>

File: src/warehouse_robot_description/urdf/warehouse_robot.urdf.xacro (robot description, xacro)
@@ -12,4 +12,8 @@
 <xacro:property name="lidar_radius" value="0.04"/>
 <xacro:property name="lidar_height" value="0.05"/>
+<!-- Camera dimensions -->
+<xacro:property name="camera_width" value="0.04"/>
+<xacro:property name="camera_height" value="0.03"/>
+<xacro:property name="camera_depth" value="0.03"/>
   <!-- ================= BASE ================= -->
   <link name="base_link">
@@ -56,4 +60,31 @@
   <inertial>
     <mass value="0.2"/>
+    <origin xyz="0 0 0"/>
+    <inertia
+      ixx="0.0001"
+      ixy="0"
+      ixz="0"
+      iyy="0.0001"
+      iyz="0"
+      izz="0.0001"/>
+  </inertial>
+</link>
+<!-- ================= Camera ================= -->
+<link name="camera_link">
+  <visual>
+    <geometry>
+      <box size="${camera_depth} ${camera_width} ${camera_height}"/>
+    </geometry>
+    <material name="Black">
+      <color rgba="0.1 0.1 0.1 1"/>
+    </material>
+  </visual>
+  <collision>
+    <geometry>
+      <box size="${camera_depth} ${camera_width} ${camera_height}"/>
+    </geometry>
+  </collision>
+  <inertial>
+    <mass value="0.1"/>
     <origin xyz="0 0 0"/>
     <inertia
@@ -193,3 +224,13 @@
         rpy="0 0 0"/>
 </joint>
+<!-- ================= Camera Joint ================= -->
+<joint
+    name="camera_joint"
+    type="fixed">
+    <parent link="base_link"/>
+    <child link="camera_link"/>
+    <origin
+        xyz="0.15 0 0.12"
+        rpy="0 0 0"/>
+</joint>
 </robot>
